File: sch/power.sch (KiCad schematic (older format))
At the start: 33 parts, among them P8 LiFePo4, P9 Button_on, Q1 Q_PMOS_GSD, Q2 Q_PMOS_GSD, Q3 Q_NMOS_DSG, U6 STMPS2141STR, U7 MCP73123, U8 LT1613, U9 NCP1450

Commit message: power done
Parts:
- added C33: 0.22uF, symbol C
- added R23: 5.1k, symbol R
- added R24, R26: 10k, symbol R
- added R25: shunt, symbol R
- added U10, U11: INA138, symbol INA138
- added U12: 74LVC1G32, symbol 74LVC1G32
- added U13: 74LVC1G17, symbol 74LVC1G17
- added U14: 74LVC2G74, symbol 74LVC2G74
- added U15: 74LVC1G02, symbol 74LVC1G02
- R11: value 20k -> Rl
- R12, R13, R19, R20: value 5.1k -> 1k
- R21: value 1k -> 5.1k
- R22: value shunt -> Rl
Connections:
- net Iuin0 is gone; now on net VCC: Q1.2 (S), R12.2, R14.2
- net +3V3: now also U10.5 (V+), U11.5 (V+); no longer R11.2
- net BOOST5V_EN: now also R21.2, U12.1
- net CHRG_EN: now also R23.2, U12.2
- net GND: now also R11.2, R21.1, R22.2, C33.2, R23.1, R24.2, R26.2, U10.2 (GND), U11.2 (GND), U12.3 (GND), U13.3 (GND), U14.4 (GND), U15.3 (GND); no longer P9.1 (P1)
- net ISCH: now also R11.1, U10.1 (OUT)
- net IUIN: now also R22.1, U11.1 (OUT)
- net Isch0: now also R25.2, U10.3 (Vs+); no longer R22.2
- net Isch1: now also R25.1, U10.4 (Vs-); no longer R22.1
- net Iuin1: now also U11.4 (Vs-)
- net SHDN: now also R26.1, U15.1, U15.2; no longer R21.1
- net VUSB_IN: no longer R11.1
- net VCC: now reaches P8.1 (P1), P8.2 (P2), Q2.3 (D), R18.1, R19.2, U7.3 (Vbat), U7.4 (Vbat)
- net VCC: now also P9.2 (P2), U11.3 (Vs+), U12.5 (VCC), U13.5 (VCC), U14.2 (~CLR), U14.7 (~PRE), U14.8 (VCC), U15.5 (VCC)
- net at Q1.1 (G): now also U12.4
- new net: Q2.1 (G), U14.3 (~Q)
- new net: C33.1, P9.1 (P1), R24.1, U13.2
- new net: U13.4, U14.1 (C)
- new net: U14.2 (~CLR), U15.4
- now unconnected: R18.2
- no-connect marks 1 -> 2
Other:
- note removed: "Логическое \nИЛИ???"
- note removed: "Схема ДОЛЖНА быть отключена от питания, \nкогда работает бустер.\n\nКогда бустер не работает она МОЖЕТ быть выключена c помощью CHRG_EN"
- note removed: "при нажатии кнопки включения мосфет открыается\nи питает схему. далее мосфет держит открытым МК.\nКогда нужно выключится МК пинает ножку вверх и\nмосфет закрывается."
- moved on the sheet: P9, Q2

Commit message: footprints done
Parts:
- removed C31: 200uF, symbol C
- removed R18: 10K, symbol R
- added C18, C30: 100uF, Capacitors_ThroughHole:C_Radial_D5_L11_P2.5, symbol CP
- added C26: 0.1uF, Capacitors_SMD:C_0402, symbol C
- added C32: 220uF, Capacitors_ThroughHole:C_Radial_D5_L11_P2.5, symbol CP
- added P12: 3.3v, Pin_Headers:Pin_Header_Straight_2x02, symbol CONN_02X02
- C27: value 100uF -> 0.1uF; footprint (none) -> Capacitors_SMD:C_0402
- C28: renamed from C25; value C -> 20uF; footprint (none) -> Capacitors_SMD:C_0805
- C29: renamed from C33; footprint (none) -> Capacitors_SMD:C_0805
- C31: renamed from C26; value C -> 10uF; footprint (none) -> Capacitors_SMD:C_0805
- C33: renamed from C28; footprint (none) -> Capacitors_SMD:C_0805
- C34: renamed from C29; footprint (none) -> Capacitors_SMD:C_0805
- C35: renamed from C30; footprint (none) -> Capacitors_SMD:C_0805
- D1, D2: footprint (none) -> DO-214AC(SMA):DO-214AC(SMA)
- L1, L2, L3: footprint (none) -> Choke_SMD:Choke_SMD_Wuerth-WE-PD2-Typ-L
- P10: renamed from P9; footprint (none) -> Pin_Headers:Pin_Header_Straight_1x02
- P11: renamed from P8; footprint (none) -> Pin_Headers:Pin_Header_Straight_2x02
- Q1, Q2, Q3: footprint (none) -> TO_SOT_Packages_SMD:SOT-23
- R11: footprint (none) -> Resistors_SMD:R_0603
- R12: value 1k -> 10k; footprint (none) -> Resistors_SMD:R_0603
- R13: value 1k -> 5k; footprint (none) -> Resistors_SMD:R_0603
- R14: renamed from R21; footprint (none) -> Resistors_SMD:R_0603
- R15: renamed from R22; footprint (none) -> Resistors_SMD:R_0603
- R16: renamed from R23; footprint (none) -> Resistors_SMD:R_0603
- R17: renamed from R14; footprint (none) -> Resistors_SMD:R_2010_HandSoldering
- R18: renamed from R15; value R -> 6.2k; footprint (none) -> Resistors_SMD:R_0603
- R19: renamed from R16; value R -> 2k; footprint (none) -> Resistors_SMD:R_0805
- R20: renamed from R17; footprint (none) -> Resistors_SMD:R_0603
- R21: renamed from R24; footprint (none) -> Resistors_SMD:R_0603
- R22: renamed from R19; value 1k -> 5.1k; footprint (none) -> Resistors_SMD:R_0603
- R23: renamed from R20; value 1k -> 5.1k; footprint (none) -> Resistors_SMD:R_0603
- R24: renamed from R25; footprint (none) -> Resistors_SMD:R_1210_HandSoldering
- R25: renamed from R26; footprint (none) -> Resistors_SMD:R_0603
- U10: renamed from U6; footprint (none) -> TO_SOT_Packages_SMD:SOT-23-5
- U11: renamed from U7; footprint (none) -> Housings_DFN_QFN:DFN-10-1EP_3x3mm_Pitch0.5mm
- U12: renamed from U8; footprint (none) -> TO_SOT_Packages_SMD:SOT-23-5
- U13: footprint (none) -> TO_SOT_Packages_SMD:SOT-353
- U14: footprint (none) -> ssop8:SSOP8
- U15: footprint (none) -> TO_SOT_Packages_SMD:SOT-23-5
- U16: renamed from U9; footprint (none) -> TO_SOT_Packages_SMD:SOT-23-5
- U7: renamed from U10; footprint (none) -> TO_SOT_Packages_SMD:SOT-23-5
- U8: renamed from U11; footprint (none) -> TO_SOT_Packages_SMD:SOT-23-5
- U9: renamed from U12; footprint (none) -> TO_SOT_Packages_SMD:SOT-323
Connections:
- net +3V3: now also C27.1, C26.1, P12.1 (P1); no longer C33.1, C35.1, D2.1 (K), U16.2 (OUT)
- net GND: now also C18.2, C26.2, C30.2, C32.2, P12.2 (P2), P12.4 (P4)
- net Isch1: now also R22.2, C18.1; no longer C27.1
- net VCC: now also C30.1; no longer R22.2
- net SHDN_IRQ: now reaches U13.4, U14.1 (C)
- new net: C32.1, C33.1, C35.1, D2.1 (K), P12.3 (P3), U16.2 (OUT)
Other:
- moved on the sheet: R22, R23

Commit message: layout 60%
Parts:
- added C36: 100uF, Capacitors_ThroughHole:C_Radial_D5_L11_P2.5, symbol CP
- R13: value 5k -> 10k
- R17: footprint Resistors_SMD:R_2010_HandSoldering -> Resistors_SMD:R_2010
- R24: footprint Resistors_SMD:R_1210_HandSoldering -> Resistors_SMD:R_2010
- U13: symbol 74LVC1G17 -> 74LVC1G17-RESCUE-sch
- U14: symbol 74LVC2G74 -> 74LVC2G74-RESCUE-sch
- U15: symbol 74LVC1G02 -> 74LVC1G02-RESCUE-sch
- U9: footprint TO_SOT_Packages_SMD:SOT-323 -> TO_SOT_Packages_SMD:SOT-353; symbol 74LVC1G32 -> 74LVC1G32-RESCUE-sch
Connections:
- net GND: now also C36.2
- net VUSB_IN: now also C36.1
- net at U14.2 (D): now also C30.1, P10.2 (P2), P11.1 (P1), P11.2 (P2), Q2.3 (D), U11.3 (Vbat), U11.4 (Vbat), U13.5 (VCC), U14.7 (~PRE), U14.8 (VCC), U15.5 (VCC); no longer U15.4
- removed net VCC: C30.1, P10.2 (P2), P11.1 (P1), P11.2 (P2), Q1.2 (S), Q2.3 (D), R12.2, R17.2, U11.3 (Vbat), U11.4 (Vbat), U13.5 (VCC), U14.2 (~CLR), U14.7 (~PRE), U14.8 (VCC), U15.5 (VCC), U8.3 (Vs+), U9.5 (VCC)
- new net: U14.6 (~CLR), U15.4
- new net Iuin0: Q1.2 (S), R12.2, R17.2, U8.3 (Vs+), U9.5 (VCC)
