File: sch/sch.kicad_pcb (KiCad board)
At the start: 2 copper layers, 9 parts, among them P1 CONN_01X09, U1 STM32F401RETx, U2 gl8088se, U3 LSM303D

Commit message: footprints done
Parts:
- removed BT1: Battery, Connect:QMS-1X52-SMD
- removed GS1: GS2, Connect:Banana_Jack_3Pin
- added C10: 0.1uF, Capacitors_SMD:C_0402, F.Cu at (177.6, 94.5)
- added C11: 1uF, Capacitors_SMD:C_0805, F.Cu at (176.4, 82.2)
- added C12: 0.1uF, Capacitors_SMD:C_0402, F.Cu at (201.5, 69.4)
- added C13: 22pF, Capacitors_SMD:C_0805, F.Cu at (185.2, 75.8)
- added C14: 22pF, Capacitors_SMD:C_0805, F.Cu at (193.6, 67.5)
- added C15: 4.7uF, Capacitors_SMD:C_0805, F.Cu at (180.8, 82.2)
- added C16: 22pF, Capacitors_SMD:C_0805, F.Cu at (168.4, 94.5)
- added C17: 22pF, Capacitors_SMD:C_0805, F.Cu at (203.3, 57.2)
- added C18: 100uF, Capacitors_ThroughHole:C_Radial_D5_L11_P2.5, F.Cu at (158.4, 120.5)
- added C19: 15uF, Capacitors_SMD:C_0402, F.Cu at (201.3, 74.9)
- added C20: 0.22uF, Capacitors_SMD:C_0805, F.Cu at (163.5, 89.7)
- added C21: 1uF, Capacitors_SMD:C_0402, F.Cu at (189.6, 81.3)
- added C22: 4.7uF, Capacitors_SMD:C_0805, F.Cu at (163.0, 96.0)
- added C23: 1uF, Capacitors_SMD:C_0402, F.Cu at (197.4, 73.0)
- added C24: 10uF, Capacitors_SMD:C_0805, F.Cu at (207.6, 57.2)
- added C25: 0.1uF, Capacitors_SMD:C_0402, F.Cu at (181.0, 88.2)
- added C26: 0.1uF, Capacitors_SMD:C_0402, F.Cu at (193.8, 124.6)
- added C27: 0.1uF, Capacitors_SMD:C_0402, F.Cu at (179.9, 137.5)
- added C28: 20uF, Capacitors_SMD:C_0805, F.Cu at (176.3, 129.7)
- added C29: 0.22uF, Capacitors_SMD:C_0805, F.Cu at (191.0, 112.8)
- added C30: 100uF, Capacitors_ThroughHole:C_Radial_D5_L11_P2.5, F.Cu at (167.9, 113.9)
- added C31: 10uF, Capacitors_SMD:C_0805, F.Cu at (198.7, 105.5)
- added C32: 220uF, Capacitors_ThroughHole:C_Radial_D5_L11_P2.5, F.Cu at (178.1, 107.2)
- added C33: 0.2uF, Capacitors_SMD:C_0805, F.Cu at (183.7, 119.8)
- added C34: 10uF, Capacitors_SMD:C_0805, F.Cu at (172.0, 129.3)
- added C35: 15uF, Capacitors_SMD:C_0805, F.Cu at (168.6, 135.6)
- added C4: 4.7uF, Capacitors_SMD:C_0805, F.Cu at (203.6, 63.5)
- added C5: 0.1uF, Capacitors_SMD:C_0402, F.Cu at (172.9, 94.5)
- added C6: 0.1uF, Capacitors_SMD:C_0402, F.Cu at (185.5, 81.7)
- added C7: 0.1uF, Capacitors_SMD:C_0402, F.Cu at (206.2, 69.4)
- added C8: 0.1uF, Capacitors_SMD:C_0402, F.Cu at (196.8, 78.5)
- added C9: 0.1uF, Capacitors_SMD:C_0402, F.Cu at (185.7, 87.2)
- added CON1: SD_Card, sch:DM3D-SF, F.Cu at (47.8, 100.6)
- added D1: D_Schottky, DO-214AC(SMA):DO-214AC(SMA), F.Cu at (108.2, 123.4)
- added D2: D_Schottky, DO-214AC(SMA):DO-214AC(SMA), F.Cu at (105.2, 130.0)
- added L1: INDUCTOR, Choke_SMD:Choke_SMD_Wuerth-WE-PD2-Typ-L, F.Cu at (97.5, 137.7)
- added L2: INDUCTOR, Choke_SMD:Choke_SMD_Wuerth-WE-PD2-Typ-L, F.Cu at (107.7, 138.2)
- added L3: INDUCTOR, Choke_SMD:Choke_SMD_Wuerth-WE-PD2-Typ-L, F.Cu at (117.9, 138.2)
- added P10: Button_on, Pin_Headers:Pin_Header_Straight_1x02, F.Cu at (152.7, 122.0)
- added P11: LiFePo4, Pin_Headers:Pin_Header_Straight_2x02, F.Cu at (144.2, 122.0)
- added P12: 3.3v, Pin_Headers:Pin_Header_Straight_2x02, F.Cu at (151.3, 108.5)
- added P2: UART, Pin_Headers:Pin_Header_Straight_1x03, F.Cu at (183.1, 60.2)
- added P3: usb, Pin_Headers:Pin_Header_Angled_1x05, F.Cu at (27.9, 141.2)
- added P4: Buttons_1, Pin_Headers:Pin_Header_Straight_2x04, F.Cu at (99.1, 111.3)
- added P5: Leds_gnd, Pin_Headers:Pin_Header_Straight_1x02, F.Cu at (179.4, 74.5)
- added P6: Buttons_2, Pin_Headers:Pin_Header_Straight_2x04, F.Cu at (108.2, 111.3)
- added P7: Leds, Pin_Headers:Pin_Header_Straight_1x04, F.Cu at (173.7, 60.2)
- added P8: 3V_bat, Pin_Headers:Pin_Header_Straight_1x02, F.Cu at (187.9, 60.2)
- added P9: LCD, Pin_Headers:Pin_Header_Straight_1x09, F.Cu at (56.9, 106.7)
- added Q1: Q_PMOS_GSD, TO_SOT_Packages_SMD:SOT-23, F.Cu at (161.0, 112.3)
- added Q2: Q_PMOS_GSD, TO_SOT_Packages_SMD:SOT-23, F.Cu at (171.2, 105.7)
- added Q3: Q_NMOS_DSG, TO_SOT_Packages_SMD:SOT-23, F.Cu at (161.0, 105.7)
- added R1: 5.1k, Resistors_SMD:R_0603, F.Cu at (142.1, 79.3)
- added R11: Rl, Resistors_SMD:R_0603, F.Cu at (197.1, 118.2)
- added R12: 10k, Resistors_SMD:R_0603, F.Cu at (175.9, 135.8)
- added R13: 5k, Resistors_SMD:R_0603, F.Cu at (189.9, 118.9)
- added R14: 5.1k, Resistors_SMD:R_0603, F.Cu at (195.7, 112.3)
- added R15: Rl, Resistors_SMD:R_0603, F.Cu at (172.4, 135.4)
- added R16: 5.1k, Resistors_SMD:R_0603, F.Cu at (182.1, 125.9)
- added R17: shunt, Resistors_SMD:R_2010_HandSoldering, F.Cu at (115.8, 130.0)
- added R18: 6.2k, Resistors_SMD:R_0603, F.Cu at (199.4, 111.6)
- added R19: 2k, Resistors_SMD:R_0805, F.Cu at (164.7, 135.3)
- added R2: 5.1k, Resistors_SMD:R_0603, F.Cu at (138.4, 79.3)
- added R20: 2.2k, Resistors_SMD:R_0603, F.Cu at (185.8, 125.9)
- added R21: 10k, Resistors_SMD:R_0603, F.Cu at (180.1, 131.8)
- added R22: 5.1k, Resistors_SMD:R_0603, F.Cu at (193.5, 118.9)
- added R23: 5.1k, Resistors_SMD:R_0603, F.Cu at (189.6, 124.8)
- added R24: shunt, Resistors_SMD:R_1210_HandSoldering, F.Cu at (89.4, 130.0)
- added R25: 10k, Resistors_SMD:R_0603, F.Cu at (183.5, 131.8)
- added R3: 5.1k, Resistors_SMD:R_0603, F.Cu at (147.8, 92.6)
- added R4: 5.1k, Resistors_SMD:R_0603, F.Cu at (189.1, 75.6)
- added R7: 330, Resistors_SMD:R_0603, F.Cu at (197.4, 67.3)
- added R8: 330, Resistors_SMD:R_0603, F.Cu at (192.7, 75.6)
- added SW1: SW_PUSH, Buttons_Switches_SMD:SW_SPST_PTS645, F.Cu at (32.0, 101.6)
- added U10: STMPS2141STR, TO_SOT_Packages_SMD:SOT-23-5, F.Cu at (138.6, 133.0)
- added U11: MCP73123, Housings_DFN_QFN:DFN-10-1EP_3x3mm_Pitch0.5mm, F.Cu at (186.6, 106.0)
- added U12: LT1613, TO_SOT_Packages_SMD:SOT-23-5, F.Cu at (177.3, 123.2)
- added U13: 74LVC1G17, TO_SOT_Packages_SMD:SOT-353, F.Cu at (164.2, 120.1)
- added U14: 74LVC2G74, ssop8:SSOP8, F.Cu at (100.6, 123.4)
- added U15: 74LVC1G02, TO_SOT_Packages_SMD:SOT-23-5, F.Cu at (149.0, 137.8)
- added U16: NCP1450, TO_SOT_Packages_SMD:SOT-23-5, F.Cu at (96.5, 131.1)
- added U4: LSM303D, sch:LGA-16-3x3, F.Cu at (72.1, 117.3)
- added U5: gl8088se, Air_Coils_SML_NEOSID:Neosid_Air-Coil_SML_2turn_HDM0231A, F.Cu at (111.8, 98.6)
- added U6: GPS_ANTENNA, sch:GSP_ANTENNA, F.Cu at (102.6, 96.5)
- added U7: INA138, TO_SOT_Packages_SMD:SOT-23-5, F.Cu at (185.3, 113.2)
- added U8: INA138, TO_SOT_Packages_SMD:SOT-23-5, F.Cu at (193.8, 106.0)
- added U9: 74LVC1G32, TO_SOT_Packages_SMD:SOT-323, F.Cu at (137.1, 139.5)
- added Y1: 8MHz, Crystals:Crystal_SMD_5032_4Pads, F.Cu at (31.0, 113.8)
- added Y2: 32768, Crystals:Crystal_Round_Horizontal_2mm, F.Cu at (178.3, 63.5)
- C1: value 15uF -> 10uF; footprint Capacitors_SMD:C_0402 -> Capacitors_SMD:C_0805
- C2: value 1uF -> 0.1uF
- C3: value 1uF -> 1nF
- P1: value CONN_01X09 -> SWD; footprint Pin_Headers:Pin_Header_Straight_1x09 -> Pin_Headers:Pin_Header_Straight_1x03
- U1: value STM32F401RETx -> 24C512; footprint Housings_QFP:LQFP-64-1EP_10x10mm_Pitch0.5mm -> SMD_Packages:SOIC-8-N
- U2: value gl8088se -> STM32F401RETx; footprint Air_Coils_SML_NEOSID:Neosid_Air-Coil_SML_2turn_HDM0231A -> Housings_QFP:LQFP-64_10x10mm_Pitch0.5mm
- U3: value LSM303D -> 74HC595; footprint sch:LGA-16-3x3 -> Housings_SOIC:SOIC-16_3.9x9.9mm_Pitch1.27mm
- moved U2 186.3 mm to (45.7, 118.4)
- moved U1 119.4 mm to (86.9, 137.7)
- moved U3 95.0 mm to (117.3, 115.3)
- moved P1 74.7 mm to (147.9, 82.5)
- moved C3 49.4 mm to (211.3, 56.8)
- moved C1 47.2 mm to (176.5, 88.5)
- moved C2 45.5 mm to (208.3, 63.1)
Connections:
- net /G_RX0 renamed Net-(U2-Pad1)
- net /G_TX0 renamed Net-(U2-Pad2)
- C3 pad 1: Net-(BT1-Pad1) -> GND
- C3 pad 2: GND -> /SWCLK
- P1 pad 1: /L_MISO -> /SWCLK
- P1 pad 2: /L_LED -> GND
- P1 pad 3: /L_SCK -> /SWDIO
- U1 pad 1: Net-(U1-Pad1) -> GND
- U1 pad 2: Net-(U1-Pad2) -> GND
- U1 pad 3: Net-(U1-Pad3) -> GND
- U1 pad 4: Net-(U1-Pad4) -> GND
- U1 pad 5: Net-(U1-Pad5) -> /I2C1_SDA
- U1 pad 6: Net-(U1-Pad6) -> /I2C1_SCL
- U1 pad 7: Net-(U1-Pad7) -> GND
- U1 pad 8: Net-(U1-Pad8) -> +3V3
- U3 pad 1: (no net) -> Net-(P7-Pad2)
- U3 pad 10: (no net) -> +3V3
- U3 pad 11: (no net) -> /K_CLK
- U3 pad 12: (no net) -> /K_LATCH
- U3 pad 13: (no net) -> GND
- U3 pad 14: (no net) -> /K_DAT
- U3 pad 15: (no net) -> Net-(P7-Pad1)
- U3 pad 16: (no net) -> +3V3
- U3 pad 2: (no net) -> Net-(P7-Pad3)
- U3 pad 3: (no net) -> Net-(P7-Pad4)
- U3 pad 4: (no net) -> Net-(P4-Pad8)
- U3 pad 5: (no net) -> Net-(P4-Pad6)
- U3 pad 6: (no net) -> Net-(P4-Pad4)
- U3 pad 7: (no net) -> Net-(P4-Pad2)
- U3 pad 8: (no net) -> GND
- U3 pad 9: (no net) -> Net-(U3-Pad9)
Other:
- board outline added: 98.6 x 49.8 mm

Commit message: layout 60%
Parts:
- removed CON1: SD_Card, sch:DM3D-SF
- added C36: 100uF, Capacitors_ThroughHole:C_Radial_D5_L11_P2.5, B.Cu at (66.9, 138.0)
- added P13: CONN_01X02, Pin_Headers:Pin_Header_Straight_1x02, F.Cu at (27.1, 135.5)
- added R5: 50, Resistors_SMD:R_0603, F.Cu at (94.5, 95.8)
- added REF**: 1pin, Connect:1pin, F.Cu at (112.2, 140.7)
- added REF**: 1pin, Connect:1pin, F.Cu at (112.2, 96.1)
- added REF**: 1pin, Connect:1pin, F.Cu at (27.4, 96.0)
- added REF**: 1pin, Connect:1pin, F.Cu at (27.4, 140.7)
- added U17: microSD, sch:DM3D-SF, F.Cu at (52.3, 129.2)
- L1, L2, L3, P12, U6: moved to B.Cu
- P4: value Buttons_1 -> btns1; footprint Pin_Headers:Pin_Header_Straight_2x04 -> Pin_Headers:Pin_Header_Straight_1x02
- P6: value Buttons_2 -> btns2; footprint Pin_Headers:Pin_Header_Straight_2x04 -> Pin_Headers:Pin_Header_Straight_1x04
- R13: value 5k -> 10k
- R17: footprint Resistors_SMD:R_2010_HandSoldering -> Resistors_SMD:R_2010
- R24: footprint Resistors_SMD:R_1210_HandSoldering -> Resistors_SMD:R_2010
- U5: value gl8088se -> ML8088se; footprint Air_Coils_SML_NEOSID:Neosid_Air-Coil_SML_2turn_HDM0231A -> sch:ML8088sE
- U9: footprint TO_SOT_Packages_SMD:SOT-323 -> TO_SOT_Packages_SMD:SOT-353
- moved C7 174.5 mm to (37.4, 113.8), turned to 90 degrees
- moved C3 169.3 mm to (52.0, 114.4), turned to 90 degrees
- moved C14 161.3 mm to (35.0, 97.0), turned to 90 degrees
- moved C17 157.5 mm to (50.9, 96.7)
- moved C8 156.7 mm to (41.7, 101.0)
- moved C4 155.2 mm to (54.0, 104.6), turned to 270 degrees
- moved C9 150.4 mm to (36.4, 105.8), turned to 90 degrees
- moved C12 150.3 mm to (53.8, 97.2), turned to 90 degrees
- moved P2 149.7 mm to (56.8, 140.5), turned to 90 degrees
- moved C15 149.4 mm to (34.6, 112.9), turned to 270 degrees
- moved C2 147.0 mm to (72.9, 120.4)
- moved C24 142.2 mm to (76.7, 112.8), turned to 270 degrees
- moved C13 141.6 mm to (45.1, 96.2), turned to 270 degrees
- moved C6 135.6 mm to (52.0, 105.3), turned to 270 degrees
- moved Y2 134.3 mm to (48.1, 96.3), turned to 90 degrees
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Connections:
- C30 pad 1: +3V3 -> Net-(C30-Pad1)
- P10 pad 2: +3V3 -> Net-(C30-Pad1)
- P11 pad 1: +3V3 -> Net-(C30-Pad1)
- P11 pad 2: +3V3 -> Net-(C30-Pad1)
- P3 pad 2: /U_ID -> /U_DP
- P3 pad 3: /U_DP -> /U_DM
- P3 pad 4: /U_DM -> /U_ID
- P4 pad 2: Net-(P4-Pad2) -> /K_BUT2
- P6 pad 1: /K_BUT2 -> Net-(P6-Pad1)
- P6 pad 2: Net-(P4-Pad2) -> Net-(P6-Pad2)
- P6 pad 3: /K_BUT2 -> Net-(P6-Pad3)
- P6 pad 4: Net-(P4-Pad4) -> Net-(P6-Pad4)
- Q1 pad 2: +3V3 -> /Sheet5813F141/Iuin0
- Q2 pad 3: +3V3 -> Net-(C30-Pad1)
- R12 pad 2: +3V3 -> /Sheet5813F141/Iuin0
- R17 pad 2: +3V3 -> /Sheet5813F141/Iuin0
- U11 pad 3: +3V3 -> Net-(C30-Pad1)
- U11 pad 4: +3V3 -> Net-(C30-Pad1)
- U13 pad 5: +3V3 -> Net-(C30-Pad1)
- U14 pad 2: Net-(U14-Pad2) -> Net-(C30-Pad1)
- U14 pad 6: (no net) -> Net-(U14-Pad6)
- U14 pad 7: +3V3 -> Net-(C30-Pad1)
- U14 pad 8: +3V3 -> Net-(C30-Pad1)
- U15 pad 4: Net-(U14-Pad2) -> Net-(U14-Pad6)
- U15 pad 5: +3V3 -> Net-(C30-Pad1)
- U2 pad 29: Net-(U2-Pad29) -> /SPEAK
- U2 pad 37: /G_RX1 -> /D_RX
- U2 pad 38: /G_TX1 -> /D_TX
- U2 pad 58: /D_RX -> /G_RX1
- U2 pad 59: /D_TX -> /G_TX1
- U3 pad 4: Net-(P4-Pad8) -> Net-(P6-Pad1)
- U3 pad 5: Net-(P4-Pad6) -> Net-(P6-Pad2)
- U3 pad 6: Net-(P4-Pad4) -> Net-(P6-Pad3)
- U3 pad 7: Net-(P4-Pad2) -> Net-(P6-Pad4)
- U6 pad 1: Net-(U5-Pad22) -> Net-(R5-Pad1)
- U6 pad 2: Net-(U5-Pad21) -> Net-(R5-Pad2)
- U6 pad 3: Net-(U5-Pad20) -> Net-(R5-Pad1)
- U8 pad 3: +3V3 -> /Sheet5813F141/Iuin0
Routing:
- net GND: track 0.00 -> 581.4 mm, vias 0 -> 9
- net +3V3: track 0.00 -> 267.8 mm, vias 0 -> 8
- net /Sheet5813F141/SHDN: track 0.00 -> 114.9 mm, vias 0 -> 8
- net /Sheet5813F141/SHDN_IRQ: track 0.00 -> 105.6 mm, vias 0 -> 4
- net /Sheet5813F141/UFAULT: track 0.00 -> 94.8 mm, vias 0 -> 4
- net /Sheet5813F141/CH_STAT: track 0.00 -> 94.7 mm, vias 0 -> 6
- net /Sheet5813F141/VUIN: track 0.00 -> 88.1 mm, vias 0 -> 6
- net /Sheet5813F141/ISCH: track 0.00 -> 86.9 mm, vias 0 -> 6
- net /Sheet5813F141/VUSB_IN: track 0.00 -> 78.2 mm, vias 0 -> 3
- net /Sheet5813F141/BOOST5V_EN: track 0.00 -> 75.5 mm, vias 0 -> 7
- net /Sheet5813F141/IUIN: track 0.00 -> 70.0 mm, vias 0 -> 8
- net /Sheet5813F141/Isch1: track 0.00 -> 66.8 mm, vias 0 -> 3
- net /Sheet5813F141/VBAT: track 0.00 -> 64.4 mm, vias 0 -> 6
- net /D_TX: track 0.00 -> 55.2 mm, vias 0 -> 3
- net /D_RX: track 0.00 -> 53.1 mm, vias 0 -> 4
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Other:
- outline, holes or cut-outs redrawn

Commit message: pcb 100%
Parts:
- moved C11 55.1 mm to (111.9, 120.2)
- moved C21 19.9 mm to (94.6, 104.9), turned to 90 degrees
- moved C20 19.3 mm to (61.1, 107.7)
- moved C22 15.9 mm to (66.7, 104.5), turned to 180 degrees
- moved R3 15.5 mm to (73.2, 122.0), turned to 180 degrees
- moved C25 13.9 mm to (68.6, 110.7)
- moved C19 13.8 mm to (93.3, 110.2), turned to 0 degrees
- moved R4 12.8 mm to (70.5, 123.8)
- moved C24 10.3 mm to (69.6, 105.3)
- moved C10 8.14 mm to (82.2, 116.5)
- moved U6 3.62 mm to (102.4, 96.5), turned to 0 degrees
- moved C26 3.52 mm to (82.1, 121.2), turned to 0 degrees
- moved P10 2.96 mm to (103.4, 123.4)
- moved C2 2.69 mm to (70.2, 120.6), turned to 270 degrees
- moved R7 1.35 mm to (105.4, 117.5), turned to 180 degrees
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Connections:
- U4 pad 7: Net-(U4-Pad7) -> +3V3
Routing:
- net GND: track 581.4 -> 828.7 mm, vias 9 -> 26
- net +3V3: track 267.8 -> 476.9 mm, vias 8 -> 17
- net /K_BUT2: track 9.13 -> 86.4 mm, vias 1 -> 4
- net /K_BUT1: track 5.79 -> 76.4 mm, vias 1 -> 4
- net /G_RST: track 2.84 -> 63.0 mm, vias 1 -> 4
- net /I2C1_SDA: track 0.00 -> 52.0 mm, vias 0 -> 6
- net /K_DAT: track 0.00 -> 49.5 mm, vias 0 -> 2
- net /K_LATCH: track 0.00 -> 47.8 mm, vias 0 -> 2
- net /K_CLK: track 0.00 -> 45.9 mm, vias 0 -> 2
- net Net-(R5-Pad1): track 0.00 -> 44.6 mm, vias 0 -> 2
- net /I2C1_SCL: track 0.00 -> 37.9 mm, vias 0 -> 5
- net /G_TX1: track 0.00 -> 36.9 mm, vias 0 -> 2
- net /G_RX1: track 0.00 -> 36.0 mm, vias 0 -> 2
- net /C_INT1: track 5.36 -> 40.5 mm, vias 1 -> 2
- net /C_RES: track 5.61 -> 38.9 mm, vias 1 -> 2
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- added copper zone on B.Cu, net GND
- added copper zone on F.Cu, net GND
- added copper zone on B.Cu, net Net-(R5-Pad1)
- added copper zone on F.Cu, net Net-(R5-Pad1)

Commit message: name on pcb
Other:
- board text added: "2016"
- board text added: "Alexander"
- board text added: "Lutsai"
- board text added: "svelotracker"
- board text added: "svelotracker by Alexander Lutsai. nov 2016 V001"
- board text added: "v001"
Changed lines of the file:
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@@
     (area 9.526001 80.685196 150.280252 151.083001)
     (thickness 1.6)
-    (drawings 11)
+    (drawings 17)
     (tracks 1906)
     (zones 0)
@@
     )
   )
+  (gr_text Lutsai (at 68.453 97.536) (layer F.Cu)
+    (effects (font (size 1.5 1.5) (thickness 0.3)))
+  )
+  (gr_text v001 (at 77.978 112.3315) (layer F.Cu)
+    (effects (font (size 1.5 1.5) (thickness 0.3)))
+  )
+  (gr_text 2016 (at 77.7875 114.427) (layer F.Cu)
+    (effects (font (size 1.5 1.5) (thickness 0.3)))
+  )
+  (gr_text Alexander (at 69.6595 95.377) (layer F.Cu)
+    (effects (font (size 1.5 1.5) (thickness 0.3)))
+  )
+  (gr_text svelotracker (at 65.3415 101.5365) (layer F.Cu)
+    (effects (font (size 1.5 1.5) (thickness 0.3)))
+  )
+  (gr_text "svelotracker by Alexander Lutsai. nov 2016 V001" (at 59.436 95.631) (layer B.Cu)
+    (effects (font (size 1.5 1.5) (thickness 0.3)) (justify mirror))
+  )
   (dimension 89.979522 (width 0.3) (layer Dwgs.User)
     (gr_text "89,980 mm" (at 69.889692 82.185196 359.9595654) (layer Dwgs.User)
@@
     (connect_pads (clearance 0.2))
     (min_thickness 0.2)
-    (fill (arc_segments 16) (thermal_gap 0.508) (thermal_bridge_width 0.508))
+    (fill yes (arc_segments 16) (thermal_gap 0.508) (thermal_bridge_width 0.508))
     (polygon
       (pts
@@
     (connect_pads (clearance 0.2))
     (min_thickness 0.2)
-    (fill (arc_segments 16) (thermal_gap 0.508) (thermal_bridge_width 0.508))
+    (fill yes (arc_segments 16) (thermal_gap 0.508) (thermal_bridge_width 0.508))
     (polygon
       (pts
@@
     (connect_pads (clearance 0.2))
     (min_thickness 0.2)
-    (fill (arc_segments 16) (thermal_gap 0.508) (thermal_bridge_width 0.508))
+    (fill yes (arc_segments 16) (thermal_gap 0.508) (thermal_bridge_width 0.508))
     (polygon
       (pts
@@
     (connect_pads (clearance 0.2))
     (min_thickness 0.2)
-    (fill (arc_segments 16) (thermal_gap 0.508) (thermal_bridge_width 0.508))
+    (fill yes (arc_segments 16) (thermal_gap 0.508) (thermal_bridge_width 0.508))
     (polygon
       (pts

Commit message: pcb ready. gerber files also.
Parts:
- added C37: 0.1uF, Capacitors_SMD:C_0402, B.Cu at (46.2, 130.0)
- added P14: RESET, Pin_Headers:Pin_Header_Straight_1x02, F.Cu at (51.3, 101.4)
- added P15: GPS_UART0, Pin_Headers:Pin_Header_Straight_1x02, B.Cu at (85.2, 96.8)
- C11: moved to B.Cu
- C19: footprint Capacitors_SMD:C_0402 -> Capacitors_SMD:C_0805
- P13: value CONN_01X02 -> SPEAKR
- U6: moved to F.Cu
- moved C11 69.0 mm to (43.3, 127.8), turned to 90 degrees
- moved R5 5.73 mm to (98.7, 100.6)
- moved U6 1.54 mm to (101.2, 95.5)
- moved C19 0.55 mm to (93.8, 110.2)
Connections:
- U5 pad 20: Net-(R5-Pad1) -> Net-(U5-Pad20)
- U5 pad 22: Net-(R5-Pad1) -> Net-(U5-Pad20)
- U6 pad 1: Net-(R5-Pad1) -> Net-(U5-Pad20)
- U6 pad 2: Net-(R5-Pad2) -> Net-(R5-Pad1)
- U6 pad 3: Net-(R5-Pad1) -> Net-(U5-Pad20)
Routing:
- net Net-(R5-Pad1): track 44.6 -> 4.35 mm, vias 2 -> 0
- net Net-(U5-Pad20): track 0.00 -> 36.6 mm
- net Net-(P15-Pad1): track 0.00 -> 11.4 mm, vias 0 -> 1
- net GND: track 828.7 -> 838.8 mm, vias 26 -> 28
- net Net-(P15-Pad2): track 0.00 -> 7.62 mm, vias 0 -> 1
- net +3V3: track 476.9 -> 481.3 mm, vias 17 -> 18
- net Net-(C12-Pad1): track 23.6 -> 25.7 mm
- net /Sheet5813F141/VUIN: track 88.1 -> 89.8 mm
- net /Sheet5813F141/ISCH: track 86.9 -> 88.4 mm
- net /K_BUT1: track 76.4 -> 75.8 mm
- net (no net): track 0.71 -> 0.16 mm
- net Net-(R5-Pad2): track 11.3 -> 11.2 mm, vias 1 -> 0
- added copper zone on F.Cu, net Net-(U5-Pad20)
- removed copper zone on B.Cu, net Net-(R5-Pad1)
- removed copper zone on F.Cu, net Net-(R5-Pad1)
Other:
- board text added: "nov 2016 V001"
- board text added: "svelotracker by Alexander Lutsai"
- board text removed: "svelotracker by Alexander Lutsai. nov 2016 V001"
