File: sch/sch.sch (KiCad schematic (older format))
At the start: 52 parts, among them CON1 SD_Card, P1 CONN_01X09, P2 Buttons_1, P3 Leds_gnd, P4 Buttons_2, P5 Leds, P6 WakeUp Button, P7 USB_OTG, SW1 SW_PUSH, U1 STM32F401RETx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

Commit message: power done
Parts:
- added C32: 1nF, symbol C_Small
- added P10: SWD, symbol CONN_01X03
- added P11: UART, symbol CONN_01X03
- P7: symbol USB_OTG -> USB_OTG-RESCUE-sch
Connections:
- net labels added: D_TX, P_5VEN, P_CHEN, P_SHDN, P_UFLT, S_D0, S_D1, S_D2, S_D3
- net labels removed: C_CS, P_BOOST5V, P_CHRG, S_DAT0, S_DAT1, S_DAT2, S_DAT3
- wire segments 326 -> 277
- no-connect marks 10 -> 13
Other:
- moved on the sheet: U3

Commit message: footprints done
Parts:
- removed BT1: Battery, Connect:QMS-1X52-SMD, symbol Battery
- removed C24: 100nF, symbol C
- removed GS1: GS2, Connect:Banana_Jack_3Pin, symbol GS2
- removed P6: WakeUp Button, symbol CONN_01X02
- removed P7: USB_OTG, symbol USB_OTG-RESCUE-sch
- removed R10: 100, symbol R
- removed R3, R4: 330, symbol R
- removed R9: 10k, symbol R
- added P3: usb, Pin_Headers:Pin_Header_Angled_1x05, symbol CONN_01X05
- added P8: 3V_bat, Pin_Headers:Pin_Header_Straight_1x02, symbol CONN_01X02
- added U6: GPS_ANTENNA, sch:GSP_ANTENNA, symbol GPS_ANTENNA
- C1: renamed from C8; footprint (none) -> Capacitors_SMD:C_0805
- C10: renamed from C16; footprint (none) -> Capacitors_SMD:C_0402
- C11: renamed from C17; footprint (none) -> Capacitors_SMD:C_0805
- C12: renamed from C18; footprint (none) -> Capacitors_SMD:C_0402
- C13: renamed from C19; footprint (none) -> Capacitors_SMD:C_0805
- C14: renamed from C20; footprint (none) -> Capacitors_SMD:C_0805
- C15: renamed from C21; footprint (none) -> Capacitors_SMD:C_0805
- C16: renamed from C22; footprint (none) -> Capacitors_SMD:C_0805
- C17: renamed from C23; footprint (none) -> Capacitors_SMD:C_0805
- C2: renamed from C9; footprint (none) -> Capacitors_SMD:C_0402
- C20: renamed from C4; footprint (none) -> Capacitors_SMD:C_0805
- C22: renamed from C5; value C -> 4.7uF; footprint (none) -> Capacitors_SMD:C_0805
- C24: renamed from C6; footprint (none) -> Capacitors_SMD:C_0805
- C25: renamed from C7; footprint (none) -> Capacitors_SMD:C_0402
- C3: renamed from C32; footprint (none) -> Capacitors_SMD:C_0402
- C4: renamed from C10; footprint (none) -> Capacitors_SMD:C_0805
- C5: renamed from C11; footprint (none) -> Capacitors_SMD:C_0402
- C6: renamed from C12; footprint (none) -> Capacitors_SMD:C_0402
- C7: renamed from C13; footprint (none) -> Capacitors_SMD:C_0402
- C8: renamed from C14; footprint (none) -> Capacitors_SMD:C_0402
- C9: renamed from C15; footprint (none) -> Capacitors_SMD:C_0402
- CON1: footprint 10067847-001 -> sch:DM3D-SF
- P1: renamed from P10; footprint (none) -> Pin_Headers:Pin_Header_Straight_1x03
- P2: renamed from P11; footprint (none) -> Pin_Headers:Pin_Header_Straight_1x03
- P4: renamed from P2; footprint (none) -> Pin_Headers:Pin_Header_Straight_2x04
- P5: renamed from P3; footprint (none) -> Pin_Headers:Pin_Header_Straight_1x02
- P6: renamed from P4; footprint (none) -> Pin_Headers:Pin_Header_Straight_2x04
- P7: renamed from P5; footprint (none) -> Pin_Headers:Pin_Header_Straight_1x04
- P9: renamed from P1; value CONN_01X09 -> LCD
- R1, R2: footprint (none) -> Resistors_SMD:R_0603
- R3: renamed from R7; footprint (none) -> Resistors_SMD:R_0603
- R4: renamed from R8; footprint (none) -> Resistors_SMD:R_0603
- R7: renamed from R5; footprint (none) -> Resistors_SMD:R_0603
- R8: renamed from R6; footprint (none) -> Resistors_SMD:R_0603
- SW1: footprint (none) -> Buttons_Switches_SMD:SW_SPST_PTS645
- U1: renamed from U5; footprint (none) -> SMD_Packages:SOIC-8-N
- U2: renamed from U1; footprint Housings_QFP:LQFP-64-1EP_10x10mm_Pitch0.5mm -> Housings_QFP:LQFP-64_10x10mm_Pitch0.5mm
- U3: renamed from U4; footprint (none) -> Housings_SOIC:SOIC-16_3.9x9.9mm_Pitch1.27mm
- Y1: footprint (none) -> Crystals:Crystal_SMD_5032_4Pads
- Y2: footprint (none) -> Crystals:Crystal_Round_Horizontal_2mm
- renumbered C1 to C19, C2 to C21, C3 to C23, U3 to U4, U2 to U5
Connections:
- net GND: now also R7.1, R8.1, P3.1 (P1), P8.2 (P2); no longer P5.1 (P1), P5.2 (P2)
- net U_DM: now also P3.4 (P4)
- net U_DP: now also P3.3 (P3)
- net U_ID: now also P3.2 (P2)
- net U_VBUS: now also P3.5 (P5)
- net at C23.1, U5.12 (V_RTC): now also P8.1 (P1)
- net at U5.20 (RF_GND): now also U6.3 (GND); no longer U5.22 (RF_GND)
- net at U5.21 (IN_RF): now also U6.2 (FEED)
- net at U3.1 (QB): now also P7.2 (P2); no longer R7.1
- net at U3.15 (QA): now also P7.1 (P1); no longer R8.1
- net at U3.2 (QC): now also P7.3 (P3)
- net at U3.3 (QD): now also P7.4 (P4)
- net at R8.2: now also P5.2 (P2); no longer P7.1 (P1)
- net at R7.2: now also P5.1 (P1); no longer P7.2 (P2)
- new net: U5.22 (RF_GND), U6.1 (GND)
Other:
- moved on the sheet: P5, P7, R7, R8

Commit message: layout 60%
Parts:
- removed CON1: SD_Card, sch:DM3D-SF, symbol SD_Card
- removed P4: Buttons_1, Pin_Headers:Pin_Header_Straight_2x04, symbol CONN_02X04
- removed P6: Buttons_2, Pin_Headers:Pin_Header_Straight_2x04, symbol CONN_02X04
- added P13: CONN_01X02, Pin_Headers:Pin_Header_Straight_1x02, symbol CONN_01X02
- added P4: btns1, Pin_Headers:Pin_Header_Straight_1x02, symbol CONN_01X02
- added P6: btns2, Pin_Headers:Pin_Header_Straight_1x04, symbol CONN_01X04
- added R5: 50, Resistors_SMD:R_0603, symbol R
- added U17: microSD, sch:DM3D-SF, symbol microSD
- U3: symbol 74HC595 -> 74HC595-RESCUE-sch
- U5: value gl8088se -> ML8088se; footprint Air_Coils_SML_NEOSID:Neosid_Air-Coil_SML_2turn_HDM0231A -> sch:ML8088sE
Connections:
- net +3V3: now also U17.4 (VDD)
- net D_RX: now also U2.37 (PC6/I2S2_MCK/SDIO_D6/TIM3_CH1/USART6_TX); no longer U2.58 (I2C1_SCL/TIM4_CH1/USART1_TX/PB6)
- net D_TX: now also U2.38 (PC7/I2S3_MCK/SDIO_D7/TIM3_CH2/USART6_RX); no longer U2.59 (I2C1_SDA/TIM4_CH2/USART1_RX/PB7)
- net GND: now also P13.1 (P1), U17.6 (VSS)
- net G_RX1: now also U2.58 (I2C1_SCL/TIM4_CH1/USART1_TX/PB6); no longer U2.37 (PC6/I2S2_MCK/SDIO_D6/TIM3_CH1/USART6_TX)
- net G_TX1: now also U2.59 (I2C1_SDA/TIM4_CH2/USART1_RX/PB7); no longer U2.38 (PC7/I2S3_MCK/SDIO_D7/TIM3_CH2/USART6_RX)
- net K_BUT1: now also P4.1 (P1)
- net K_BUT2: now also P4.2 (P2)
- net S_CLK: now also U17.5 (CLK)
- net S_CMD: now also U17.3 (CMD)
- net S_D0: now also U17.7 (DAT0)
- net S_D1: now also U17.8 (DAT1)
- net S_D2: now also U17.1 (DAT2)
- net S_D3: now also U17.2 (DAT3)
- net U_DM: now also P3.3 (P3); no longer P3.4 (P4)
- net U_DP: now also P3.2 (P2); no longer P3.3 (P3)
- net U_ID: now also P3.4 (P4); no longer P3.2 (P2)
- net SPEAK: now reaches U2.29 (I2C2_SCL/I2S2_CK/SPI2_SCK/TIM2_CH3/PB10)
- net SPEAK: now also P13.2 (P2)
- net at U5.20 (RF_GND), U6.3 (GND): now also U5.22 (RF_GND), U6.1 (GND), R5.1
- net at U5.21 (IN_RF), U6.2 (FEED): now also R5.2
- net at U3.4 (QE): now also P6.1 (P1)
- net at U3.5 (QF): now also P6.2 (P2)
- net at U3.6 (QG): now also P6.3 (P3)
- net at U3.7 (QH): now also P6.4 (P4)
- no-connect marks 13 -> 12
Other:
- moved on the sheet: R1

Commit message: pcb 100%
Connections:
- net +3V3: now also U4.7 (SDO)
- no-connect marks 12 -> 11
Changed lines of the file:
@@
 Text Label 7900 4350 0    60   ~ 0
 G_RST
-NoConn ~ 9000 1300
 NoConn ~ 3250 4150
 Text Label 2900 3050 0    60   ~ 0
@@
 Wire Wire Line
 	3650 6200 3650 6900
+Wire Wire Line
+	9000 1300 8900 1300
+Wire Wire Line
+	8900 1300 8900 1400
+Connection ~ 8900 1400
 $EndSCHEMATC

Commit message: pcb ready. gerber files also.
Parts:
- added C37: 0.1uF, Capacitors_SMD:C_0402, symbol C
- added P14: RESET, Pin_Headers:Pin_Header_Straight_1x02, symbol CONN_01X02
- added P15: GPS_UART0, Pin_Headers:Pin_Header_Straight_1x02, symbol CONN_01X02
- C19: footprint Capacitors_SMD:C_0402 -> Capacitors_SMD:C_0805
- P13: value CONN_01X02 -> SPEAKR
Connections:
- net +3V3: now also C37.1
- net GND: now also C37.2, P14.1 (P1)
- net at C12.1, SW1.2, U2.7 (NRST): now also P14.2 (P2)
- net at U5.1 (RX0): now also P15.2 (P2)
- net at U5.2 (TX0): now also P15.1 (P1)
- net at U5.20 (RF_GND), U5.22 (RF_GND), U6.1 (GND)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: no longer R5.1
- net at R5.2, U5.21 (IN_RF): no longer U6.2 (FEED)
- new net: R5.1, U6.2 (FEED)
- no-connect marks 11 -> 9
Other:
- moved on the sheet: R5, U6
